Commit message: Trying to add robot model using stl. It seems to be working. I now need to create a better model based on the one found online.

File: bebop_description/urdf/bebop_base.urdf.xacro (robot description, xacro)
@@ -12,5 +12,13 @@
   <xacro:property name="tilt_vel" value="2.0" />
   <xacro:property name="joint_effort" value="50" />
-  <link name="base_link"></link>
+  <link name="base_link">
+    <visual>
+      <origin rpy="0 0 1.5708" xyz="0.0 0 0.0"/>
+      <geometry>
+<!--	<box size="0.38 0.036 0.33" />-->
+        <mesh size ="0.1 0.1 0.1" filename="package://bebop_description/meshes/bebop_chassis2.stl"/>
+      </geometry>
+    </visual>
+  </link>
   <link name="camera_base_link"></link>
   <link name="camera_pan_link"></link>

Commit message: New bebop model! It's so cool now!

File: bebop_description/urdf/bebop_base.urdf.xacro (robot description, xacro)
@@ -17,5 +17,5 @@
       <geometry>
 <!--	<box size="0.38 0.036 0.33" />-->
-        <mesh size ="0.1 0.1 0.1" filename="package://bebop_description/meshes/bebop_chassis2.stl"/>
+        <mesh size ="0.1 0.1 0.1" filename="package://bebop_description/meshes/bebop.stl"/>
       </geometry>
     </visual>
